Commit message: Edited Rt Xacro. Added build bash script for xacro->urdf

File: allegro_hand_description/allegro_hand_description_left.xacro (robot description, xacro)
@@ -1,4 +1,4 @@
 <?xml version="1.0"?>
-<robot xmlns:xacro="http://www.ros.org/wiki/xacro" name="AllegroHand_Left">
+<robot xmlns:xacro="http://www.ros.org/wiki/xacro" name="allegro_hand_left">
 <xacro:property name="DEG2RAD" value="0.01745329251" />
 <!-- ======================== BASE PARAMS ========================= -->

File: allegro_hand_description/allegro_hand_description_right.urdf (robot description, URDF)
Before this commit: robot AllegroHand_Left, 21 links, 20 joints
Joints:
- joint joint_12.0: limit lower=-1 upper=1 effort=0 velocity=0 -> lower=0.263 upper=1.396 effort=0 velocity=0

File: allegro_hand_description/allegro_hand_description_right.xacro (robot description, xacro)
@@ -1,4 +1,4 @@
 <?xml version="1.0"?>
-<robot xmlns:xacro="http://www.ros.org/wiki/xacro" name="AllegroHand_Left">
+<robot xmlns:xacro="http://www.ros.org/wiki/xacro" name="allegro_hand_right">
 <!--
 rosrun xacro xacro.py allegro_hand_description_right.urdf.xacro > allegro_hand_description_right.urdf
@@ -158,6 +158,5 @@
   <joint name="joint_${finger_num*4+0}" type="revolute">
     <axis xyz="-1 0 0"/>
-    <!--<limit effort="0" velocity="0" lower="${limit_0_t_low-joint_safety_margin}" upper="${limit_0_t_up-joint_safety_margin}" />-->
-    <limit effort="0" velocity="0" lower="-1" upper="1" />
+    <limit effort="0" velocity="0" lower="${limit_0_t_low-joint_safety_margin}" upper="${limit_0_t_up-joint_safety_margin}" />
     <parent link="base_link"/>
     <child link="link_${finger_num*4+0}"/>
