Commit message: Left URDF finished. Bash build fixed.

File: allegro_hand_description/allegro_hand_description_right.xacro (robot description, xacro)
@@ -19,4 +19,8 @@
 <xacro:property name="link3_z" value="0.0387" />
 <xacro:property name="fingerTip_r" value="0.0120" />
+<xacro:property name="offset_origin_x_const" value="0" />
+<xacro:property name="offset_origin_y_const" value="0.0435" /> <!--0.0435,   0.044981-->
+<xacro:property name="offset_origin_z_const" value="-0.001542" /> <!--0.002298-->
+<xacro:property name="offset_origin_z_mid_const" value="0.0007" /> <!--0.002298-->
 <!-- ========================= THUMB PARAMS ========================= -->
 <xacro:property name="link0_t_x" value="0.0358" />
@@ -48,30 +52,26 @@
 <!-- ============================================================================= -->
 <!-- BASE -->
-  <link name="base_link">
-    <visual>
-      <geometry>
-      	<mesh filename="package://allegro_hand_description/meshes/base_link.STL" />
-      	<!--     drawing  estimate  estimate  -->
-        <!--<box size="0.0408 0.1130 ${base_link_z}"/> -->
-      </geometry>
-      <!--<origin rpy="0 0 0" xyz="-0.009300 0 -${base_link_z/2}"/>-->
-      <material name="black">
-        <color rgba="0.2 0.2 0.2 1"/>
-      </material>
-    </visual>
+<link name="base_link">
+	<visual>
+    	<geometry>
+      		<mesh filename="package://allegro_hand_description/meshes/base_link.STL" />
+      	</geometry>
+      	<!-- LEFT -->
+      	<!-- <origin rpy="${-90*DEG2RAD} 0 0" xyz="0 0 0 "/> -->
+      	<!-- RIGHT -->
+      	<origin rpy="0 0 0" xyz="0 0 0 "/>
+      	<material name="black">
+        	<color rgba="0.2 0.2 0.2 1"/>
+      	</material>
+	</visual>
     <collision>
-      <geometry>
-      	<!--     drawing  estimate  estimate  -->
-        <box size="0.0408 0.1130 ${base_link_z}"/>
-      </geometry>
-		<origin rpy="0 0 0" xyz="-0.009300 0 -${base_link_z/2}"/>
+	    <origin rpy="0 0 0" xyz="-0.009300 0 -${base_link_z/2}"/>
+    	<geometry>
+        	<box size="0.0408 0.1130 ${base_link_z}"/>
+      	</geometry>
     </collision>
   </link>
 <!-- ============================================================================= -->
 <!-- FINGERS -->
-<xacro:property name="offset_origin_x_const" value="0" />
-<xacro:property name="offset_origin_y_const" value="0.0435" /> <!--0.0435,   0.044981-->
-<xacro:property name="offset_origin_z_const" value="-0.001542" /> <!--0.002298-->
-<xacro:property name="offset_origin_z_mid_const" value="0.0007" /> <!--0.002298-->
 <!-- RIGHT HAND due to which finger is number 0 -->
 <!-- for LEFT HAND switch the sign of the **offset_origin_y** and **finger_angle_r** parameters-->
@@ -97,4 +97,5 @@
 	finger_angle_r=		"${5.0*DEG2RAD}"
 />
+<!-- THUMB -->
 <xacro:thumb_right
 	finger_num=			"3"
@@ -106,412 +107,258 @@
 	finger_angle_y=		"-${90*DEG2RAD}"
 />
-	<!-- offset_origin_z=	"-0.07308"
-		finger_num=			"3"
-	offset_origin_x=	"-0.0182"
-	offset_origin_y=	"0.019333"
-	offset_origin_z=	"-0.044987"
-	-->
-	<!-- THE STL ORIGIN NEEDS TO BE FIXED. ALSO THESE NUMBERS NEED TO BE DERIVEDFROM DRAWING, NOT SOLIDOWRKS EXP URDF, see the drawing on the wiki -->
 <!--
 <xacro:thumb_left
 	finger_num=			"3"
 	offset_origin_x=	"-0.0182"
-	offset_origin_y=	"-0.0168753"
-	offset_origin_z=	"-0.07308"
-	finger_angle_r=		"0"
+	offset_origin_y=	"-0.019333"
+	offset_origin_z=	"-0.045987"
+	finger_angle_r=		"${90*DEG2RAD}"
 	finger_angle_p=		"-${95*DEG2RAD}"
 	finger_angle_y=		"${90*DEG2RAD}"
 />
 -->
-<!-- -${95*DEG2RAD}    ${180*DEG2RAD} -->
-<!-- ============================================================================= -->
-<!-- LEFT -->
-<!-- THUMB -->
-<!-- Write code for left and right with proper changes
-	(using variables for like comps) and include as 2 macros
-	include both and comment unused for right and left -->
-<!-- END LEFT -->
-<!-- ============================================================================= -->
-<!-- ============================================================================= -->
-<!-- ============================================================================= -->
-<!-- THUMB MACROS -->
+<!-- ============================================================================= -->
+<!-- ============================================================================= -->
+<!-- ============================================================================= -->
+<!-- THUMB MACRO -->
 <xacro:macro name="thumb_right" params="finger_num offset_origin_x offset_origin_y offset_origin_z finger_angle_r finger_angle_p finger_angle_y">
-<!-- [LINK 0] [LINK 0] [LINK 0] [LINK 0]  [LINK 0] [LINK 0] [LINK 0] -->
+<!-- [LINK 12] -->
 	<link name="link_${finger_num*4+0}">
-    <visual>
-      <geometry>
-        <!--<box size="${link0_t_x} ${link0_t_y} ${link0_t_z}"/>-->
-      	<mesh filename="package://allegro_hand_description/meshes/link_12.0_left.STL" />
-      </geometry>
-      <!--<origin rpy="0 0 0" xyz="${-0.0358/2+0.027} ${0.034/2-0.026} ${0.045/2-0.008}"/>-->
-      <material name="black">
-        <color rgba=".2 .2 .2 1"/>
-      </material>
-    </visual>
-    <collision>
-      <geometry>
-        <box size="${link0_t_x} ${link0_t_y} ${link0_t_z}"/>
-      </geometry>
-      <origin rpy="0 0 0" xyz="${-0.0358/2+0.027} ${0.034/2-0.026} ${0.045/2-0.008}"/>
-    </collision>
-  </link>
-  <joint name="joint_${finger_num*4+0}" type="revolute">
-    <axis xyz="-1 0 0"/>
-    <limit effort="0" velocity="0" lower="${limit_0_t_low-joint_safety_margin}" upper="${limit_0_t_up-joint_safety_margin}" />
-    <parent link="base_link"/>
-    <child link="link_${finger_num*4+0}"/>
-    <origin rpy="${finger_angle_r} ${finger_angle_p} ${finger_angle_y}" xyz="${offset_origin_x} ${offset_origin_y} ${offset_origin_z}"/>
+    	<visual>
+			<geometry>
+        		<!-- RIGHT -->
+      			<mesh filename="package://allegro_hand_description/meshes/link_12.0_right.STL" />
+      			<!-- LEFT -->
+      			<!-- <mesh filename="package://allegro_hand_description/meshes/link_12.0_left.STL" /> -->
+      		</geometry>
+      		<material name="black">
+        		<color rgba=".2 .2 .2 1"/>
+      		</material>
+    	</visual>
+    	<collision>
+      		<geometry>
+        		<box size="${link0_t_x} ${link0_t_y} ${link0_t_z}"/>
+      		</geometry>
+  			<!-- RIGHT -->
+            <origin rpy="0 0 0" xyz="${-0.0358/2+0.0} ${.018/2} ${.029/2}"/>
+     		<!-- LEFT -->
+     		<!-- <origin rpy="0 0 0" xyz="${-0.0358/2+0.0} ${-.018/2} ${.029/2}"/> -->
+    	</collision>
+	</link>
+	<joint name="joint_${finger_num*4+0}" type="revolute">
+    	<axis xyz="-1 0 0"/>
+    	<limit effort="0" velocity="0" lower="${limit_0_t_low-joint_safety_margin}" upper="${limit_0_t_up-joint_safety_margin}" />
+    	<parent link="base_link"/>
+    	<child link="link_${finger_num*4+0}"/>
+    	<origin rpy="${finger_angle_r} ${finger_angle_p} ${finger_angle_y}" xyz="${offset_origin_x} ${offset_origin_y} ${offset_origin_z}"/>
+	</joint>
+<!-- [LINK 13] -->
+	<link name="link_${finger_num*4+1}">
+		<visual>
+			<geometry>
+		    	<mesh filename="package://allegro_hand_description/meshes/link_13.0.STL" />
+		  	</geometry>
+		  	<material name="black">
+		  		<color rgba=".2 .2 .2 1"/>
+		 	</material>
+		</visual>
+		<collision>
+			<geometry>
+		    	<box size="${links_x} ${links_y} ${link1_t_z}"/>
+		  	</geometry>
+		  	<origin rpy="0 0 0" xyz="0 0 ${link1_t_z/2}"/>
+		</collision>
+	</link>
+  	<joint name="joint_${finger_num*4+1}" type="revolute">
+    	<axis xyz="0 0 1"/>
+     	<limit effort="0" velocity="0" lower="${limit_1_t_low+joint_safety_margin}" upper="${limit_1_t_up-joint_safety_margin}" />
+    	<parent link="link_${finger_num*4+0}"/>
+    	<child link="link_${finger_num*4+1}"/>
+		<!-- RIGHT -->
+    	<origin xyz="-0.027 0.005 0.0399"/>
+    	<!-- LEFT -->
+    	<!-- <origin xyz="-0.027 -0.005 0.0399"/> -->
+  	</joint>
+<!-- [LINK 14] -->
+	<link name="link_${finger_num*4+2}">
+		<visual>
+			<geometry>
+		  		<mesh filename="package://allegro_hand_description/meshes/link_14.0.STL" />
+			</geometry>
+			<material name="black">
+		  	</material>
+		</visual>
+		<collision>
+			<geometry>
+		    	<box size="${links_x} ${links_y} ${link2_t_z}"/>
+		  	</geometry>
+		  	<origin rpy="0 0 0" xyz="0 0 ${link2_t_z/2}"/>
+		</collision>
+	</link>
+  <joint name="joint_${finger_num*4+2}" type="revolute">
+		<axis xyz="0 1 0"/>
+		<limit effort="0" velocity="0" lower="${limit_2_t_low+joint_safety_margin}" upper="${limit_2_t_up-joint_safety_margin}" />
+		<parent link="link_${finger_num*4+1}"/>
+		<child link="link_${finger_num*4+2}"/>
+		<origin xyz="0 0 ${link1_t_z}"/>
   </joint>
-<!-- [LINK 1] [LINK 1] [LINK 1] [LINK 1]  [LINK 1] [LINK 1] [LINK 1] -->
-	<link name="link_${finger_num*4+1}">
-    <visual>
-      <geometry>
-        <!--<box size="${links_x} ${links_y} ${link1_t_z}"/>-->
-      	<mesh filename="package://allegro_hand_description/meshes/link_13.0.STL" />
-      </geometry>
-      <!--<origin rpy="0 0 0" xyz="0 0 ${link1_t_z/2}"/>-->
-      <material name="black">
-      </material>
-    </visual>
-    <collision>
-      <geometry>
-        <box size="${links_x} ${links_y} ${link1_t_z}"/>
-      </geometry>
-      <origin rpy="0 0 0" xyz="0 0 ${link1_t_z/2}"/>
-    </collision>
-  </link>
-  <joint name="joint_${finger_num*4+1}" type="revolute">
-    <axis xyz="0 0 1"/>
-     <limit effort="0" velocity="0" lower="${limit_1_t_low+joint_safety_margin}" upper="${limit_1_t_up-joint_safety_margin}" />
-    <parent link="link_${finger_num*4+0}"/>
-    <child link="link_${finger_num*4+1}"/>
-    <!--<origin xyz="0 0 ${0.0552-0.0177}"/>-->
-    <origin xyz="-0.027 0.005 0.0399"/>
-  </joint>
-<!-- [LINK 2] [LINK 2] [LINK 2] [LINK 2]  [LINK 2] [LINK 2] [LINK 2] -->
-	<link name="link_${finger_num*4+2}">
-    <visual>
-      <geometry>
-      	<mesh filename="package://allegro_hand_description/meshes/link_14.0.STL" />
-        <!--<box size="${links_x} ${links_y} ${link2_t_z}"/>-->
-      </geometry>
-      <!--<origin rpy="0 0 0" xyz="0 0 ${link2_t_z/2}"/>-->
-      <material name="black">
-      </material>
-    </visual>
-    <collision>
-      <geometry>
-        <box size="${links_x} ${links_y} ${link2_t_z}"/>
-      </geometry>
-      <origin rpy="0 0 0" xyz="0 0 ${link2_t_z/2}"/>
-    </collision>
-  </link>
-  <joint name="joint_${finger_num*4+2}" type="revolute">
-    <axis xyz="0 1 0"/>
-     <limit effort="0" velocity="0" lower="${limit_2_t_low+joint_safety_margin}" upper="${limit_2_t_up-joint_safety_margin}" />
-    <parent link="link_${finger_num*4+1}"/>
-    <child link="link_${finger_num*4+2}"/>
-    <origin xyz="0 0 ${link1_t_z}"/>
-  </joint>
-<!-- [LINK 3] [LINK 3] [LINK 3] [LINK 3]  [LINK 3] [LINK 3] [LINK 3] -->
+<!-- [LINK 15] -->
 	<link name="link_${finger_num*4+3}">
-    <visual>
-      <geometry>
-      	<mesh filename="package://allegro_hand_description/meshes/link_15.0.STL" />
-        <!--<box size="${links_x} ${links_y} ${link3_t_z-fingerTip_r}"/>-->
-      </geometry>
-      <!--<origin rpy="0 0 0" xyz="0 0 ${(link3_t_z-fingerTip_r)/2}"/>-->
-      <material name="black">
-      </material>
-    </visual>
-    <collision>
-      <geometry>
-        <box size="${links_x} ${links_y} ${link3_t_z-fingerTip_r}"/>
-      </geometry>
-      <origin rpy="0 0 0" xyz="0 0 ${(link3_t_z-fingerTip_r)/2}"/>
-    </collision>
-  </link>
-  <joint name="joint_${finger_num*4+3}" type="revolute">
-    <axis xyz="0 1 0"/>
-     <limit effort="0" velocity="0" lower="${limit_3_t_low+joint_safety_margin}" upper="${limit_3_t_up-joint_safety_margin}" />
-    <parent link="link_${finger_num*4+2}"/>
-    <child link="link_${finger_num*4+3}"/>
-    <origin xyz="0 0 ${link2_t_z}"/>
-  </joint>
+    	<visual>
+      		<geometry>
+      				<mesh filename="package://allegro_hand_description/meshes/link_15.0.STL" />
+        	</geometry>
+    	<material name="black">
+    	</material>
+    	</visual>
+    	<collision>
+			<geometry>
+		    	<box size="${links_x} ${links_y} ${link3_t_z-fingerTip_r}"/>
+		  	</geometry>
+		  	<origin rpy="0 0 0" xyz="0 0 ${(link3_t_z-fingerTip_r)/2}"/>
+    	</collision>
+	</link>
+	<joint name="joint_${finger_num*4+3}" type="revolute">
+    	<axis xyz="0 1 0"/>
+     	<limit effort="0" velocity="0" lower="${limit_3_t_low+joint_safety_margin}" upper="${limit_3_t_up-joint_safety_margin}" />
+    	<parent link="link_${finger_num*4+2}"/>
+    	<child link="link_${finger_num*4+3}"/>
+    	<origin xyz="0 0 ${link2_t_z}"/>
+	</joint>
 <!-- [FINGER TIP] -->
 	<link name="link_${finger_num*4+3}_tip">
-    <visual>
-      <geometry>
-      	<mesh filename="package://allegro_hand_description/meshes/link_15.0_tip.STL" />
-        <!--<sphere radius="${fingerTip_r}"/>-->
-      </geometry>
-      <!--<origin rpy="0 0 0" xyz="0 0 ${link3_t_z-fingerTip_r}"/>-->
-      <material name="white">
-        <color rgba=".9 .9 .9 1"/>
-      </material>
-    </visual>
-    <collision>
-      <geometry>
-        <sphere radius="${fingerTip_r}"/>
-      </geometry>
-      <origin rpy="0 0 0" xyz="0 0 0"/>
-    </collision>
-  </link>
-  <joint name="joint_${finger_num*4+3}_tip" type="fixed">
-    <parent link="link_${finger_num*4+3}"/>
-    <child link="link_${finger_num*4+3}_tip"/>
-    <origin rpy="0 0 0" xyz="0 0 ${link3_t_z-fingerTip_r}"/> <!--0.0267000000000005-->
-  </joint>
+		<visual>
+			<geometry>
+		  		<mesh filename="package://allegro_hand_description/meshes/link_15.0_tip.STL" />
+		  	</geometry>
+		  	<material name="white">
+		  		<color rgba=".9 .9 .9 1"/>
+		  	</material>
+    	</visual>
+    	<collision>
+      		<geometry>
+        		<sphere radius="${fingerTip_r}"/>
+      		</geometry>
+      		<origin rpy="0 0 0" xyz="0 0 0"/>
+    	</collision>
+	</link>
+  	<joint name="joint_${finger_num*4+3}_tip" type="fixed">
+    	<parent link="link_${finger_num*4+3}"/>
+    	<child link="link_${finger_num*4+3}_tip"/>
+    	<origin rpy="0 0 0" xyz="0 0 ${link3_t_z-fingerTip_r}"/> <!--0.0267000000000005-->
+  	</joint>
 </xacro:macro>
-<!-- NOT USING CORRECT MESHES -->
-<xacro:macro name="thumb_left" params="finger_num offset_origin_x offset_origin_y offset_origin_z finger_angle_r finger_angle_p finger_angle_y">
-<!-- [LINK 0] [LINK 0] [LINK 0] [LINK 0]  [LINK 0] [LINK 0] [LINK 0] -->
+<!-- END THUMB MACRO -->
+<!-- THREE FINGER MACRO -->
+<xacro:macro name="finger" params="finger_num offset_origin_x offset_origin_y offset_origin_z finger_angle_r">
+<!-- [LINK 0, 4, 8] -->
 	<link name="link_${finger_num*4+0}">
-    <visual>
-      <geometry>
-        <!--<box size="${link0_t_x} ${link0_t_y} ${link0_t_z}"/>-->
-      	<mesh filename="package://allegro_hand_description/meshes/link_12.0.STL" />
-      </geometry>
-      <!--<origin rpy="0 0 0" xyz="${-0.0358/2+0.027} ${0.034/2-0.026} ${0.045/2-0.008}"/>-->
-      <material name="black">
-        <color rgba=".2 .2 .2 1"/>
-      </material>
-    </visual>
-    <collision>
-      <geometry>
-        <box size="${link0_t_x} ${link0_t_y} ${link0_t_z}"/>
-      </geometry>
-      <origin rpy="0 0 0" xyz="${-0.0358/2+0.027} ${0.034/2-0.026} ${0.045/2-0.008}"/>
-    </collision>
-  </link>
-  <joint name="joint_${finger_num*4+0}" type="revolute">
-    <axis xyz="1 0 0"/>
-     <limit effort="0" velocity="0" lower="${limit_0_t_low-joint_safety_margin}" upper="${limit_0_t_up-joint_safety_margin}" />
-    <parent link="base_link"/>
-    <child link="link_${finger_num*4+0}"/>
-    <origin rpy="${finger_angle_r} ${finger_angle_p} ${finger_angle_y}" xyz="${offset_origin_x} ${offset_origin_y} ${offset_origin_z}"/>
-  </joint>
-<!-- [LINK 1] [LINK 1] [LINK 1] [LINK 1]  [LINK 1] [LINK 1] [LINK 1] -->
+    	<visual>
+    		<geometry>
+      			<mesh filename="package://allegro_hand_description/meshes/link_0.0.STL" />
+      		</geometry>
+      		<material name="black"/>
+    	</visual>
+    	<collision>
+      		<geometry>
+        		<box size="${links_x} ${links_y} ${link0_z}"/>
+      		</geometry>
+      		<origin rpy="0 0 0" xyz="0 0 ${link0_z/2}"/>
+    	</collision>
+	</link>
+  	<joint name="joint_${finger_num*4+0}" type="revolute">
+    	<axis xyz="0 0 1"/>
+    	<limit effort="0" velocity="0" lower="${limit_0_low+joint_safety_margin}" upper="${limit_0_up-joint_safety_margin}" />
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